Commit message: change robot structure and project architecture

File: arm_description/urdf/arm.urdf.xacro (robot description, xacro)
@@ -30,7 +30,7 @@
             <mass value="${mass}" />
             <inertia ixx="${mass * (sy * sy + sz * sz) / 12}"
-                     iyy="${mass * (sx * sx + sz * sz) / 12}"
-                     izz="${mass * (sx * sx + sy * sy) / 12}"
-                     ixy="0" ixz="0" iyz="0" />
+                iyy="${mass * (sx * sx + sz * sz) / 12}"
+                izz="${mass * (sx * sx + sy * sy) / 12}"
+                ixy="0" ixz="0" iyz="0" />
         </inertial>
     </xacro:macro>
@@ -47,7 +47,7 @@
             <mass value="${mass}" />
             <inertia ixx="${mass * (3 * radius * radius + length * length) / 12}"
-                     iyy="${mass * (3 * radius * radius + length * length) / 12}"
-                     izz="${mass * radius * radius / 2}"
-                     ixy="0" ixz="0" iyz="0" />
+                iyy="${mass * (3 * radius * radius + length * length) / 12}"
+                izz="${mass * radius * radius / 2}"
+                ixy="0" ixz="0" iyz="0" />
         </inertial>
     </xacro:macro>
@@ -79,5 +79,5 @@
         </visual>
         <xacro:cylinder_physics mass="${base_mass}" radius="0.1"
-                                length="${base_height}" xyz="0 0 ${base_height / 2}" />
+            length="${base_height}" xyz="0 0 ${base_height / 2}" />
     </link>
     <!-- The joint frame is at the top of the stationary base. -->
@@ -96,16 +96,40 @@
             <origin xyz="0.04 0 ${pedestal_height / 2}" rpy="0 0 0" />
             <geometry>
-                <box size="0.14 0.08 ${pedestal_height}" />
+                <box size="0.28 0.08 ${pedestal_height}" />
             </geometry>
             <material name="orange" />
         </visual>
-        <xacro:box_physics mass="${pedestal_mass}" sx="0.14" sy="0.08"
-                           sz="${pedestal_height}" xyz="0.04 0 ${pedestal_height / 2}" />
-    </link>
+        <xacro:box_physics mass="${pedestal_mass}" sx="0.28" sy="0.08"
+            sz="${pedestal_height}" xyz="0.04 0 ${pedestal_height / 2}" />
+    </link>
+    <!-- Fixed fork supports: inner faces at Y = +/-0.028 m leave
+         3 mm clearance around the upper arm's 0.025 m radius.
+         Each block is 4 x 1.2 x 5 cm, with a provisional mass of 30 g.
+         Separate fixed links keep each block's inertia easy to understand. -->
+    <xacro:macro name="shoulder_support" params="name side">
+        <joint name="${name}_mount_joint" type="fixed">
+            <parent link="shoulder_link" />
+            <child link="${name}" />
+            <origin xyz="0.11 ${side * 0.034} ${pedestal_height + 0.025}"
+                rpy="0 0 0" />
+        </joint>
+        <link name="${name}">
+            <visual>
+                <geometry>
+                    <box size="0.04 0.012 0.05" />
+                </geometry>
+                <material name="gray" />
+            </visual>
+            <xacro:box_physics mass="0.03" sx="0.04" sy="0.012" sz="0.05"
+                xyz="0 0 0" />
+        </link>
+    </xacro:macro>
+    <xacro:shoulder_support name="left_shoulder_support_link" side="1" />
+    <xacro:shoulder_support name="right_shoulder_support_link" side="-1" />
     <!-- Shoulder pitch: local Y turns with the base rotation joint. -->
     <joint name="shoulder_joint" type="revolute">
         <parent link="shoulder_link" />
         <child link="upper_arm_link" />
-        <origin xyz="0.04 0 ${pedestal_height}" rpy="0 0 0" />
+        <origin xyz="0.11 0 ${pedestal_height + 0.025 + 0.005}" rpy="0 0 0" />
         <axis xyz="0 1 0" />
         <limit lower="${-pi / 2}" upper="${pi / 2}" effort="10" velocity="1" />
@@ -117,10 +141,13 @@
             <origin xyz="0 0 ${upper_arm_length / 2}" rpy="0 0 0" />
             <geometry>
-                <box size="0.05 0.05 ${upper_arm_length}" />
+                <cylinder radius="0.025" length="${upper_arm_length}" />
             </geometry>
             <material name="blue" />
         </visual>
-        <xacro:box_physics mass="${upper_arm_mass}" sx="0.05" sy="0.05"
-                           sz="${upper_arm_length}" xyz="0 0 ${upper_arm_length / 2}" />
+        <xacro:cylinder_physics
+            mass="${upper_arm_mass}"
+            radius="0.025"
+            length="${upper_arm_length}"
+            xyz="0 0 ${upper_arm_length / 2}" />
     </link>
     <joint name="elbow_joint" type="revolute">
@@ -136,16 +163,23 @@
             <origin xyz="0 0 ${forearm_length / 2}" rpy="0 0 0" />
             <geometry>
-                <box size="0.04 0.04 ${forearm_length}" />
+                <cylinder radius="0.02" length="${forearm_length}" />
             </geometry>
             <material name="orange" />
         </visual>
-        <xacro:box_physics mass="${forearm_mass}" sx="0.04" sy="0.04"
-                           sz="${forearm_length}" xyz="0 0 ${forearm_length / 2}" />
-    </link>
-    <!-- Fixed mounting: there is no wrist rotation joint. -->
-    <joint name="gripper_mount_joint" type="fixed">
+        <xacro:cylinder_physics
+            mass="${forearm_mass}"
+            radius="0.02"
+            length="${forearm_length}"
+            xyz="0 0 ${forearm_length / 2}" />
+    </link>
+    <!-- Wrist pitch tilts the palm and fingers independently of the elbow.
+         Zero keeps the previous straight gripper mounting; initial range +/-45 deg. -->
+    <joint name="wrist_pitch_joint" type="revolute">
         <parent link="forearm_link" />
         <child link="gripper_palm_link" />
         <origin xyz="0 0 ${forearm_length}" rpy="0 0 0" />
+        <axis xyz="0 1 0" />
+        <limit lower="${-pi / 4}" upper="${pi / 4}" effort="2" velocity="0.5" />
+        <dynamics damping="0.1" friction="0" />
     </joint>
     <link name="gripper_palm_link">
@@ -158,5 +192,5 @@
         </visual>
         <xacro:box_physics mass="${palm_mass}" sx="0.06" sy="0.10"
-                           sz="${palm_height}" xyz="0 0 ${palm_height / 2}" />
+            sz="${palm_height}" xyz="0 0 ${palm_height / 2}" />
     </link>
     <!-- The position is ONE finger's travel, in metres; total gap = 2 * position. -->
@@ -178,5 +212,5 @@
         </visual>
         <xacro:box_physics mass="${finger_mass}" sx="0.02" sy="${finger_thickness}"
-                           sz="${finger_length}" xyz="0 0 ${finger_length / 2}" />
+            sz="${finger_length}" xyz="0 0 ${finger_length / 2}" />
     </link>
     <joint name="right_finger_joint" type="prismatic">
@@ -203,5 +237,5 @@
         </visual>
         <xacro:box_physics mass="${finger_mass}" sx="0.02" sy="${finger_thickness}"
-                           sz="${finger_length}" xyz="0 0 ${finger_length / 2}" />
+            sz="${finger_length}" xyz="0 0 ${finger_length / 2}" />
     </link>
     <!-- Reference halfway along the fingers, centered in the opening. -->
@@ -213,5 +247,5 @@
     <link name="tool0" />
     <xacro:if value="$(arg gazebo)">
-        <xacro:include filename="gazebo.xacro" />
+        <xacro:include filename="$(find arm_gazebo)/urdf/gazebo.xacro" />
     </xacro:if>
 </robot>

File: arm_gazebo/urdf/gazebo.xacro (robot description, xacro)
@@ -55,4 +55,6 @@
     <xacro:position_controller joint="elbow_joint" topic="/arm/elbow/target"
                                 p="60" i="1" d="2" effort="5" />
+    <xacro:position_controller joint="wrist_pitch_joint" topic="/arm/wrist/target"
+                                p="20" i="0.5" d="1" effort="2" />
     <xacro:position_controller joint="gripper_opening_joint" topic="/arm/gripper/target"
                                 p="200" i="0.5" d="2" effort="5" />

Commit message: add camera to the gripper and adapt launch files to launch gazebo and rviz together

File: arm_description/urdf/arm.urdf.xacro (robot description, xacro)
@@ -194,4 +194,32 @@
             sz="${palm_height}" xyz="0 0 ${palm_height / 2}" />
     </link>
+    <!-- Camera beside the palm, looking along the fingers. -->
+    <joint name="camera_mount_joint" type="fixed">
+        <parent link="gripper_palm_link" />
+        <child link="camera_link" />
+        <origin xyz="0.05 0 0.01" rpy="0 ${-pi / 2} 0" />
+    </joint>
+    <link name="camera_link">
+        <visual>
+            <geometry>
+                <box size="0.03 0.04 0.02" />
+            </geometry>
+            <material name="gray" />
+        </visual>
+        <xacro:box_physics
+            mass="0.02"
+            sx="0.03"
+            sy="0.04"
+            sz="0.02"
+            xyz="0 0 0" />
+    </link>
+    <!-- Optical origin at the housing's front face. -->
+    <joint name="camera_optical_joint" type="fixed">
+        <parent link="camera_link" />
+        <child link="camera_optical_frame" />
+        <origin xyz="0.015 0 0"
+            rpy="${-pi / 2} 0 ${-pi / 2}" />
+    </joint>
+    <link name="camera_optical_frame" />
     <!-- The position is ONE finger's travel, in metres; total gap = 2 * position. -->
     <joint name="gripper_opening_joint" type="prismatic">

File: arm_gazebo/urdf/gazebo.xacro (robot description, xacro)
@@ -35,5 +35,5 @@
         <gazebo>
             <plugin filename="gz-sim-joint-position-controller-system"
-                    name="gz::sim::systems::JointPositionController">
+                name="gz::sim::systems::JointPositionController">
                 <joint_name>${joint}</joint_name>
                 <topic>${topic}</topic>
@@ -50,20 +50,43 @@
     </xacro:macro>
     <xacro:position_controller joint="base_rotation_joint" topic="/arm/base/target"
-                                p="30" i="1" d="2" effort="10" />
+        p="30" i="1" d="2" effort="10" />
     <xacro:position_controller joint="shoulder_joint" topic="/arm/shoulder/target"
-                                p="100" i="2" d="5" effort="10" />
+        p="100" i="2" d="5" effort="10" />
     <xacro:position_controller joint="elbow_joint" topic="/arm/elbow/target"
-                                p="60" i="1" d="2" effort="5" />
+        p="60" i="1" d="2" effort="5" />
     <xacro:position_controller joint="wrist_pitch_joint" topic="/arm/wrist/target"
-                                p="20" i="0.5" d="1" effort="2" />
+        p="20" i="0.5" d="1" effort="2" />
     <xacro:position_controller joint="gripper_opening_joint" topic="/arm/gripper/target"
-                                p="200" i="0.5" d="2" effort="5" />
+        p="200" i="0.5" d="2" effort="5" />
     <xacro:position_controller joint="right_finger_joint" topic="/arm/gripper/target"
-                                p="200" i="0.5" d="2" effort="5" />
+        p="200" i="0.5" d="2" effort="5" />
     <gazebo>
         <plugin filename="gz-sim-joint-state-publisher-system"
-                name="gz::sim::systems::JointStatePublisher">
+            name="gz::sim::systems::JointStatePublisher">
             <topic>/model/learning_arm/joint_state</topic>
         </plugin>
     </gazebo>
+    <!-- Sensor at the camera housing's front face. -->
+    <gazebo reference="camera_link">
+        <sensor name="wrist_camera" type="camera">
+            <pose>0.015 0 0 0 0 0</pose>
+            <always_on>true</always_on>
+            <update_rate>15</update_rate>
+            <topic>/arm/camera/image_raw</topic>
+            <camera>
+                <optical_frame_id>camera_optical_frame</optical_frame_id>
+                <camera_info_topic>/arm/camera/camera_info</camera_info_topic>
+                <horizontal_fov>1.0472</horizontal_fov>
+                <image>
+                    <width>640</width>
+                    <height>480</height>
+                    <format>R8G8B8</format>
+                </image>
+                <clip>
+                    <near>0.01</near>
+                    <far>5.0</far>
+                </clip>
+            </camera>
+        </sensor>
+    </gazebo>
 </robot>
